File: chip-hardware/chip-hardware.kicad_sch (KiCad schematic)
At the start: 22 parts

Commit message: Annotated all of the components. Everything looking good so far
Parts:
- gave numbers to parts that had none: 22
