File: chip-hardware/V3/Woodstock/Woodstock.kicad_pcb (KiCad board)
At the start: 2 copper layers, 16.5 x 19.1 mm, 11 parts, among them J1 501461-0491, U1 MCP9808_MSOP, U2 LIS3DH

Commit message: Connceted everything that needs to be connected. Looks good
Routing:
- net GND: track 0.00 -> 36.1 mm, vias 0 -> 7
- net /SDA: track 31.3 -> 34.8 mm
- net +3V3: track 103.1 -> 105.9 mm
- added copper zone on B.Cu, net GND
- added copper zone on F.Cu, net GND

Commit message: fixed all errors and removed all warnings
Routing:
- net /SDA: track 34.8 -> 34.3 mm
Other:
- outline, holes or cut-outs redrawn
Changed lines of the file:
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@@
     (property "vault revision" "5F166C2B-E9D9-4135-9ADB-F1D93D2D935E")
     (attr through_hole)
-    (fp_text reference "J1" (at -1.04084 3.16856) (layer "F.SilkS")
+    (fp_text reference "J1" (at -3.78404 -1.12404) (layer "F.SilkS")
       (effects (font (size 1 1) (thickness 0.15)) (justify right))
     )
-    (fp_text value "501461-0491" (at -0.127 0.8279 180) (layer "F.SilkS")
-      (effects (font (size 1.27 1.27) (thickness 0.15)))
+    (fp_text value "501461-0491" (at -0.02484 2.93996 180) (layer "F.SilkS")
+      (effects (font (size 0.508 0.508) (thickness 0.127)))
     )
     (fp_line (start -1.45 -0.482267) (end -1.3 -0.482267) (layer "F.SilkS") (width 0.15))
@@
     (property "Sheetname" "")
     (attr smd)
-    (fp_text reference "R3" (at 0.02596 1.40086) (layer "B.SilkS")
+    (fp_text reference "R3" (at 2.46436 -0.04694) (layer "B.SilkS")
       (effects (font (size 1 1) (thickness 0.15)) (justify mirror))
     )
@@
   (gr_circle (center 151.2062 89.662) (end 153.0604 89.8652) (layer "B.SilkS") (width 0.15) (fill none))
   (gr_circle (center 151.1554 103.8098) (end 153.0096 103.759) (layer "B.SilkS") (width 0.15) (fill none))
-  (gr_line (start 157.389938 87.301761) (end 144.752701 87.30366) (layer "Edge.Cuts") (width 0.1))
+  (gr_line (start 142.90096 104.57566) (end 142.898501 89.295422) (layer "Edge.Cuts") (width 0.1))
+  (gr_line (start 144.88216 106.42986) (end 157.533259 106.426) (layer "Edge.Cuts") (width 0.1))
   (gr_arc (start 144.88216 106.42986) (mid 143.525399 105.894001) (end 142.90096 104.57566) (layer "Edge.Cuts") (width 0.1))
-  (gr_line (start 142.90096 104.57566) (end 142.898501 89.295422) (layer "Edge.Cuts") (width 0.1))
-  (gr_line (start 144.88216 106.42986) (end 157.58216 106.426) (layer "Edge.Cuts") (width 0.1))
+  (gr_line (start 144.752701 87.30366) (end 157.389938 87.301761) (layer "Edge.Cuts") (width 0.1))
   (gr_arc (start 157.389938 87.301761) (mid 158.75056 87.83706) (end 159.3817 89.155961) (layer "Edge.Cuts") (width 0.1))
   (gr_line (start 159.387459 104.434238) (end 159.3817 89.155961) (layer "Edge.Cuts") (width 0.1))
@@
   (segment (start 149.559543 104.658662) (end 150.253559 104.658662) (width 0.2) (layer "F.Cu") (net 3))
   (segment (start 149.1704 93.519) (end 148.8694 93.218) (width 0.2) (layer "F.Cu") (net 3))
-  (segment (start 149.1704 92.7646) (end 149.1704 92.23126) (width 0.2) (layer "F.Cu") (net 3))
   (segment (start 148.329225 91.591179) (end 148.329225 92.677825) (width 0.2) (layer "F.Cu") (net 3))
   (segment (start 146.7866 93.218) (end 146.557989 92.989389) (width 0.2) (layer "F.Cu") (net 3))

Commit message: placed some additional ias
Routing:
- net GND: vias 7 -> 8
Changed lines of the file:
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@@
   (via (at 153.8478 98.5012) (size 0.8) (drill 0.4) (layers "F.Cu" "B.Cu") (free) (net 5))
   (via (at 145.796 92.2782) (size 0.8) (drill 0.4) (layers "F.Cu" "B.Cu") (net 5))
+  (via (at 151.003 100.1776) (size 0.8) (drill 0.4) (layers "F.Cu" "B.Cu") (free) (net 5))
   (via (at 148.209 102.4382) (size 0.8) (drill 0.4) (layers "F.Cu" "B.Cu") (free) (net 5))
   (via (at 144.526 89.408) (size 0.8) (drill 0.4) (layers "F.Cu" "B.Cu") (free) (net 5))

Commit message: Added adjustment to the PCB. Everything seems right
Parts:
- moved J1 1.31 mm to (150.5, 102.8), turned to 0 degrees
Routing:
- net /SDA: track 34.3 -> 41.0 mm, vias 1 -> 3
- net /SCL: track 36.4 -> 37.5 mm
- net GND: track 36.1 -> 36.8 mm
- net +3V3: track 105.9 -> 105.3 mm
