File: chip-hardware/V2/chip-hardware.kicad_pcb (KiCad board)
At the start: 2 copper layers, 62.2 x 27.4 mm, 22 parts, among them J1 KLDX-0202-B, J2 Screw_Terminal_01x02, J3 Conn_01x02, U1 TLV70033_SOT23-5, U2 LIS3DH, U3 INA260, U4 MCP9808_MSOP, U5 ESP32-WROOM-32

Commit message: Created groud planes and fixed power jack issues. Issued new gerbers for both relevant files
Changed lines of the file:
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@@
     (fp_line (start -7.4 4.65) (end -7.4 -4.65) (layer "F.Fab") (width 0.15))
     (fp_line (start 7.4 -4.65) (end 7.4 4.65) (layer "F.Fab") (width 0.15))
-    (pad "1" thru_hole rect locked (at 6.65 0 180) (size 1.4 4.899999) (drill oval 4.3) (layers *.Cu)
+    (pad "1" thru_hole rect locked (at 6.65 0 180) (size 1.4 4.899999) (drill oval 0.998 4.3) (layers *.Cu)
       (net 1 "Net-(C1-Pad1)") (pinfunction "1") (pintype "power_in"))
-    (pad "2" thru_hole roundrect locked (at 0.45 0 180) (size 1.4 4.4) (drill oval 3.8) (layers *.Cu) (roundrect_rratio 0.5)
+    (pad "2" thru_hole roundrect locked (at 0.45 0 180) (size 1.4 4.4) (drill oval 0.888 3.8) (layers *.Cu) (roundrect_rratio 0.5)
       (net 2 "GND") (pinfunction "2") (pintype "power_in"))
-    (pad "3" thru_hole roundrect locked (at 3.45 4.7 180) (size 4.4 1.4) (drill oval 0.8) (layers *.Cu) (roundrect_rratio 0.5)
+    (pad "3" thru_hole roundrect locked (at 3.45 4.7 180) (size 4.4 1.4) (drill oval 3.594 0.8) (layers *.Cu) (roundrect_rratio 0.5)
       (net 2 "GND") (pinfunction "3") (pintype "power_in"))
     (model "eec.models/Kycon_-_KLDX-0202-B.step"
